File: documentation/schematic_layout/v3/miavita.brd (EAGLE design)
At the start: 94 x 74.3 mm, 56 parts, among them IC1 REF02D, IC4 4572D, IC5 74AC590D, IC6 74LS157D, IC7 ADS1278, IC8 R3318AI, Q1 BC847B, Q2 BC847B, Q3 BC847B, Q4 BC847B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

Commit message: Small clarification in schematic
0.1f = 100uf
Parts:
- C9: value 0.1uF -> 100nF
Changed lines of the file:
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@@
 <attribute name="VALUE" x="39.878" y="10.414" size="1.27" layer="27" rot="R90"/>
 </element>
-<element name="C9" library="resistor" package="C0603" value="0.1uF" x="39.37" y="8.001" smashed="yes">
+<element name="C9" library="resistor" package="C0603" value="100nF" x="39.37" y="8.001" smashed="yes">
 <attribute name="NAME" x="41.021" y="7.493" size="1.016" layer="25"/>
 <attribute name="VALUE" x="38.481" y="5.969" size="1.27" layer="27"/>
