File: documentation/schematic_layout/v3/miavita.sch (EAGLE design)
At the start: 56 parts, among them IC1 REF02D, IC4 4572D, IC5 74AC590D, IC6 74LS157D, IC7 ADS1278, IC8 R3318AI, Q1 BC847B, Q2 BC847B, Q3 BC847B, Q4 BC847B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

Commit message: Small clarification in schematic
0.1f = 100uf
Parts:
- C9: value 0.1uF -> 100nF
Changed lines of the file:
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@@
 <part name="+3V9" library="supply1" deviceset="+3V3" device=""/>
 <part name="SUPPLY14" library="supply2" deviceset="GND" device=""/>
-<part name="C9" library="resistor" deviceset="C-EU" device="C0603" value="0.1uF"/>
+<part name="C9" library="resistor" deviceset="C-EU" device="C0603" value="100nF"/>
 <part name="SUPPLY1" library="supply2" deviceset="GND" device=""/>
 <part name="TS7500" library="con-samtec" deviceset="SSW-122-02-S-D" device=""/>
